File: CM4_HighSpeed.kicad_sch (KiCad schematic)
At the start: 8 parts, among them J10 HDMI_C_1.4, J11 HDMI_C_1.4, J8 Conn_01x22_Female, J9 Conn_01x22_Female, U7 RT9742SNGV

Commit message: Adding normal size HDMI connectors
Parts:
- J10, J11: footprint Connector_HDMI:HDMI_Micro-D_Molex_46765-0x01 -> (none)

Commit message: Adding 3D modesl
Parts:
- J10, J11: footprint (none) -> CM4IO:EDAC 690-019-298-412

Commit message: Adding audio connector - fixing USB, adding logos
Parts:
- U: renamed from J8; value Conn_01x22_Female -> (none); footprint Connector_FFC-FPC:Hirose_FH12-22S-0.5SH_1x22-1MP_P0.50mm_Horizontal -> (none)
- U: renamed from C34; value 100n -> (none); footprint Capacitor_SMD:C_0402_1005Metric -> (none)
- U: renamed from C33; value 100n -> (none); footprint Capacitor_SMD:C_0402_1005Metric -> (none)
- U: renamed from U7; value RT9742SNGV -> (none); footprint Package_TO_SOT_SMD:SOT-23 -> (none)
- U: renamed from Module1; value ComputeModule4 -> (none); footprint CM4IO:Raspberry-Pi-4-Compute-Module-noholes -> (none)
- U: renamed from J9; value Conn_01x22_Female -> (none); footprint Connector_FFC-FPC:Hirose_FH12-22S-0.5SH_1x22-1MP_P0.50mm_Horizontal -> (none)
- U: renamed from J11; value HDMI_C_1.4 -> (none); footprint CM4IO:EDAC 690-019-298-412 -> (none)
- U: renamed from J10; value HDMI_C_1.4 -> (none); footprint CM4IO:EDAC 690-019-298-412 -> (none)
Connections:
- net CAM0_C_N: no longer U.140 (CAM0_C_N)
- net CAM0_C_P: no longer U.142 (CAM0_C_P)
- net CAM0_D0_N: no longer U.128 (CAM0_D0_N)
- net CAM0_D0_P: no longer U.130 (CAM0_D0_P)
- net CAM0_D1_N: no longer U.134 (CAM0_D1_N)
- net CAM0_D1_P: no longer U.136 (CAM0_D1_P)
- net CAM1_C_N: no longer U.127 (CAM1_C_N)
- net CAM1_C_P: no longer U.129 (CAM1_C_P)
- net CAM1_D0_N: no longer U.115 (CAM1_D0_N)
- net CAM1_D0_P: no longer U.117 (CAM1_D0_P)
- net CAM1_D1_N: no longer U.121 (CAM1_D1_N)
- net CAM1_D1_P: no longer U.123 (CAM1_D1_P)
- net CAM1_D2_N: no longer U.133 (CAM1_D2_N)
- net CAM1_D2_P: no longer U.135 (CAM1_D2_P)
- net CAM1_D3_N: no longer U.139 (CAM1_D3_N)
- net CAM1_D3_P: no longer U.141 (CAM1_D3_P)
- net DSI0_C_N: no longer U.169 (DSI0_C_N)
- net DSI0_C_P: no longer U.171 (DSI0_C_P)
- net DSI0_D0_N: no longer U.157 (DSI0_D0_N)
- net DSI0_D0_P: no longer U.159 (DSI0_D0_P)
- net DSI0_D1_N: no longer U.163 (DSI0_D1_N)
- net DSI0_D1_P: no longer U.165 (DSI0_D1_P)
- net DSI1_C_N: no longer U.187 (DSI1_C_N)
- net DSI1_C_P: no longer U.189 (DSI1_C_P)
- net DSI1_D0_N: no longer U.175 (DSI1_D0_N)
- net DSI1_D0_P: no longer U.177 (DSI1_D0_P)
- net DSI1_D1_N: no longer U.181 (DSI1_D1_N)
- net DSI1_D1_P: no longer U.183 (DSI1_D1_P)
- net DSI1_D2_N: no longer U.193 (DSI1_D2_N)
- net DSI1_D2_P: no longer U.195 (DSI1_D2_P)
- net DSI1_D3_N: no longer U.194 (DSI1_D3_N)
- net DSI1_D3_P: no longer U.196 (DSI1_D3_P)
- net GND: no longer U.107 (GND), U.108 (GND), U.113 (GND), U.114 (GND), U.119 (GND), U.120 (GND), U.125 (GND), U.126 (GND), U.131 (GND), U.132 (GND), U.137 (GND), U.138 (GND), U.144 (GND), U.150 (GND), U.155 (GND), U.156 (GND), U.161 (GND), U.162 (GND), U.167 (GND), U.168 (GND), U.173 (GND), U.174 (GND), U.179 (GND), U.180 (GND), U.185 (GND), U.186 (GND), U.191 (GND), U.192 (GND), U.197 (GND), U.198 (GND)
- net HDMI0_CEC: no longer U.151 (HDMI0_CEC)
- net HDMI0_CK_N: no longer U.190 (HDMI0_CLK_N)
- net HDMI0_CK_P: no longer U.188 (HDMI0_CLK_P)
- net HDMI0_D0_N: no longer U.184 (HDMI0_TX0_N)
- net HDMI0_D0_P: no longer U.182 (HDMI0_TX0_P)
- net HDMI0_D1_N: no longer U.178 (HDMI0_TX1_N)
- net HDMI0_D1_P: no longer U.176 (HDMI0_TX1_P)
- net HDMI0_D2_N: no longer U.172 (HDMI0_TX2_N)
- net HDMI0_D2_P: no longer U.170 (HDMI0_TX2_P)
- net HDMI0_HOTPLUG: no longer U.153 (HDMI0_HOTPLUG)
- net HDMI0_SCL: no longer U.200 (HDMI0_SCL)
- net HDMI0_SDA: no longer U.199 (HDMI0_SDA)
- net HDMI1_CEC: no longer U.149 (HDMI1_CEC)
- net HDMI1_CK_N: no longer U.166 (HDMI1_CLK_N)
- net HDMI1_CK_P: no longer U.164 (HDMI1_CLK_P)
- net HDMI1_D0_N: no longer U.160 (HDMI1_TX0_N)
- net HDMI1_D0_P: no longer U.158 (HDMI1_TX0_P)
- net HDMI1_D1_N: no longer U.154 (HDMI1_TX1_N)
- net HDMI1_D1_P: no longer U.152 (HDMI1_TX1_P)
- net HDMI1_D2_N: no longer U.148 (HDMI1_TX2_N)
- net HDMI1_D2_P: no longer U.146 (HDMI1_TX2_P)
- net HDMI1_HOTPLUG: no longer U.143 (HDMI1_HOTPLUG)
- net HDMI1_SCL: no longer U.147 (HDMI1_SCL)
- net HDMI1_SDA: no longer U.145 (HDMI1_SDA)
- net PCIE_CLK_N: no longer U.112 (PCIe_CLK_N)
- net PCIE_CLK_P: no longer U.110 (PCIe_CLK_P)
- net PCIE_CLK_nREQ: no longer U.102 (PCIe_CLK_nREQ)
- net PCIE_RX_N: no longer U.118 (PCIe_RX_N)
- net PCIE_RX_P: no longer U.116 (PCIe_RX_P)
- net PCIE_TX_N: no longer U.124 (PCIe_TX_N)
- net PCIE_TX_P: no longer U.122 (PCIe_TX_P)
- net PCIE_nRST: no longer U.109 (PCIe_nRST)
- net TV_OUT: no longer U.111 (VDAC_COMP)
- net USB2_N: no longer U.103 (USB2_N)
- net USB2_P: no longer U.105 (USB2_P)
- net USBOTG_ID: no longer U.101 (USB_OTG_ID)
