File: USB2-HUB.kicad_sch (KiCad schematic)
At the start: 34 parts, among them J3 USB_OTG, J4 Conn_01x04_Male, J5 USB_A, J6 USB_A, J7 USB_MICRO, U3 FSUSB42MUX, U4 USB2514B-I/M2, U5 TPD4EUSB30, U6 AP22653W6, Y1 24MHz

Commit message: Adding audio connector - fixing USB, adding logos
Parts:
- U: renamed from R13; value 2.2K 1% -> (none); footprint Resistor_SMD:R_0402_1005Metric -> (none)
- U: renamed from C29; value 10u -> (none); footprint Capacitor_SMD:C_0805_2012Metric -> (none)
- U: renamed from C30; value 10u -> (none); footprint Capacitor_SMD:C_0805_2012Metric -> (none)
- U: renamed from C31; value 10u -> (none); footprint Capacitor_SMD:C_0805_2012Metric -> (none)
- U: renamed from C32; value 10u -> (none); footprint Capacitor_SMD:C_0805_2012Metric -> (none)
- U: renamed from R12; value 2.2K 1% -> (none); footprint Resistor_SMD:R_0402_1005Metric -> (none)
- U: renamed from U6; value AP22653W6 -> (none); footprint Package_TO_SOT_SMD:SOT-23-6 -> (none)
- U: renamed from U4; value USB2514B-I/M2 -> (none); footprint Package_DFN_QFN:QFN-36-1EP_6x6mm_P0.5mm_EP3.7x3.7mm -> (none)
- U: renamed from R16; value 36K 1% -> (none); footprint Resistor_SMD:R_0402_1005Metric -> (none)
- U: renamed from R15; value 36K 1% -> (none); footprint Resistor_SMD:R_0402_1005Metric -> (none)
- U: renamed from R14; value 36K 1% -> (none); footprint Resistor_SMD:R_0402_1005Metric -> (none)
- U: renamed from R19; value 15K 1% -> (none); footprint Resistor_SMD:R_0402_1005Metric -> (none)
- U: renamed from U3; value FSUSB42MUX -> (none); footprint Package_SO:MSOP-10_3x3mm_P0.5mm -> (none)
- U: renamed from R17; value 12K 1% -> (none); footprint Resistor_SMD:R_0402_1005Metric -> (none)
- U: renamed from R18; value 36K 1% -> (none); footprint Resistor_SMD:R_0402_1005Metric -> (none)
- U: renamed from C24; value 100n -> (none); footprint Capacitor_SMD:C_0402_1005Metric -> (none)
- U: renamed from C25; value 100n -> (none); footprint Capacitor_SMD:C_0402_1005Metric -> (none)
- U: renamed from C26; value 100n -> (none); footprint Capacitor_SMD:C_0402_1005Metric -> (none)
- U: renamed from C22; value 100n -> (none); footprint Capacitor_SMD:C_0402_1005Metric -> (none)
- U: renamed from C20; value 10u -> (none); footprint Capacitor_SMD:C_0805_2012Metric -> (none)
- U: renamed from C21; value 10u -> (none); footprint Capacitor_SMD:C_0805_2012Metric -> (none)
- U: renamed from C18; value 27pF -> (none); footprint Capacitor_SMD:C_0402_1005Metric -> (none)
- U: renamed from C19; value 27pF -> (none); footprint Capacitor_SMD:C_0402_1005Metric -> (none)
- U: renamed from C23; value 100n -> (none); footprint Capacitor_SMD:C_0402_1005Metric -> (none)
- U: renamed from C27; value 10u -> (none); footprint Capacitor_SMD:C_0805_2012Metric -> (none)
- U: renamed from U5; value TPD4EUSB30 -> (none); footprint Package_SON:USON-10_2.5x1.0mm_P0.5mm -> (none)
- U: renamed from C28; value 100uF -> (none); footprint Capacitor_Tantalum_SMD:CP_EIA-7343-31_Kemet-D -> (none)
- U: renamed from D2; value B340AE-13 -> (none); footprint Diode_SMD:D_SMB_Handsoldering -> (none)
- U: renamed from J3; value USB_OTG -> (none); footprint CM4IO:USB_Micro-B_EDAC_UCON00686 -> (none)
- U: renamed from J7; value USB_MICRO -> (none); footprint CM4IO:USB_Micro-B_EDAC_UCON00686 -> (none)
- U: renamed from Y1; value 24MHz -> (none); footprint Crystal:Crystal_SMD_EuroQuartz_X22-4Pin_2.5x2.0mm_HandSoldering -> (none)
- U: renamed from J6; value USB_A -> (none); footprint Connector_USB:USB_A_Molex_67643_Horizontal -> (none)
- U: renamed from J5; value USB_A -> (none); footprint Connector_USB:USB_A_Molex_67643_Horizontal -> (none)
- U: renamed from J4; value Conn_01x04_Male -> (none); footprint Connector_PinHeader_2.00mm:PinHeader_1x04_P2.00mm_Horizontal -> (none)
