File: kicad/Unifying.kicad_pcb (KiCad board)
At the start: 4 copper layers, 115.1 x 61 mm, 123 parts, among them J1 Conn_01x02, J10 HDMI_C_1.4, J11 HDMI_C_1.4, J12 nRpiBoot, J13 Conn_01x03, J14 Conn_01x03, J15 AudioOUT, J16 Micro_SD_Card_Det, J17 THD-20-R, J18 GLOBAL_EN, J19 AudioAMP, J2 Bus_M.2_Socket_B, J3 USB_OTG, J4 Conn_01x04_Male, J5 USB_A, J6 USB_A, J7 USB_MICRO, J8 Conn_01x22_Female, J9 Conn_01x22_Female, Q1 DMP3013SFV-7, U10 74LVC1G07SE-7, U11 RT9742GGJ5, U2 AP64501SP-13, U3 FSUSB42MUX, U4 USB2514B-I/M2, U5 TPD4EUSB30, U6 AP22653W6, U7 RT9742SNGV, U8 74LVC1G07SE-7, U9 NC7WZ16, Y1 24MHz

Commit message: Removing logo
Parts:
- removed the G*** at (152.2, 137.1)
- removed the G*** at (114.8, 108.7)

Commit message: New pictures
Parts:
- moved G*** 22.6 mm to (107.5, 135.9)
- moved REF** 16.3 mm to (123.1, 135.5)
- moved REF** 3.62 mm to (123.1, 135.4)
Changed lines of the file:
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@@
   )
   (footprint "Symbol:OSHW-Logo2_9.8x8mm_SilkScreen" locked (layer "F.Cu")
-    (at 126.61 136.2)
+    (at 123.07 135.43)
     (descr "Open Source Hardware Symbol")
     (tags "Logo Symbol OSHW")
@@
   )
   (footprint "CM4IO:balthazar-logo" locked (layer "B.Cu")
-    (at 114.17 114.29 180)
+    (at 107.47 135.86 180)
     (attr board_only exclude_from_pos_files exclude_from_bom)
     (fp_text reference "G***" (at 0 0) (layer "Dwgs.User")
@@
   )
   (footprint "Symbol:OSHW-Logo2_9.8x8mm_SilkScreen" locked (layer "B.Cu")
-    (at 114.25 121.86 180)
+    (at 123.13 135.49 180)
     (descr "Open Source Hardware Symbol")
     (tags "Logo Symbol OSHW")

Commit message: Adding power layer filled zones
Routing:
- added copper zone on In2.Cu, net /+3.3v
- added copper zone on In2.Cu, net /+3.3vSSD
- added copper zone on In2.Cu, net /+5v
- added copper zone on In2.Cu, net /USB2-HUB/VBUS
- added copper zone on In2.Cu, net Net-(J1-Pin_1)
