File: kicad/Unifying.kicad_pcb (KiCad board)
At the start: 4 copper layers, 115.1 x 61 mm, 130 parts, among them J1 Conn_01x02, J10 GPDI0, J11 GPDI1, J12 nRpiBoot, J13 Conn_01x03, J14 Conn_01x03, J15 AudioOUT, J16 Micro_SD_Card_Det, J17 THD-20-R, J18 GLOBAL_EN, J19 AudioAMP, J2 Bus_M.2_Socket_B, J20 THD-02-R, J3 USB_OTG, J4 Conn_01x04_Male, J5 USB_A, J6 USB_A, J7 USB_MICRO, J8 Conn_01x22_Female, J9 Conn_01x22_Female, Q1 DMP3013SFV-7, U1 TPD4EUSB30, U10 74LVC1G07SE-7, U11 RT9742GGJ5, U12 MagJack-A70-112-331N126, U2 AP64501SP-13, U3 FSUSB42MUX, U4 USB2514B-I/M2, U5 TPD4EUSB30, U6 AP22653W6, U7 RT9742SNGV, U8 74LVC1G07SE-7, U9 NC7WZ16, Y1 24MHz

Commit message: Adding I2S MIC connector
Parts:
- added J21: MIC, Connector_PinSocket_2.54mm:PinSocket_1x06_P2.54mm_Vertical, F.Cu at (225.2, 131.6)
Changed lines of the file:
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@@
   (net 260 "Net-(U12-LEDG_K)")
   (net 261 "Net-(U12-LEDY_K)")
+  (net 262 "/CM4_GPIO (GPIO, SDCARD)/BCLK")
+  (net 263 "/CM4_GPIO (GPIO, SDCARD)/DOUT")
+  (net 264 "/CM4_GPIO (GPIO, SDCARD)/LRCL")
+  (net 265 "/CM4_GPIO (GPIO, SDCARD)/SEL")
   (footprint "Connector_FFC-FPC:Hirose_FH12-22S-0.5SH_1x22-1MP_P0.50mm_Horizontal" (layer "F.Cu")
     (at 149.464 87.046 180)
@@
       (offset (xyz 0 0 0))
       (scale (xyz 1 1 1))
+      (rotate (xyz 0 0 0))
+    )
+  )
+  (footprint "Connector_PinSocket_2.54mm:PinSocket_1x06_P2.54mm_Vertical" (layer "F.Cu")
+    (at 225.175 131.625)
+    (descr "Through hole straight socket strip, 1x06, 2.54mm pitch, single row (from Kicad 4.0.7), script generated")
+    (tags "Through hole socket strip THT 1x06 2.54mm single row")
+    (property "Sheetfile" "File: CM4_GPIO.kicad_sch")
+    (property "Sheetname" "CM4_GPIO (GPIO, SDCARD)")
+    (property "ki_description" "Generic connector, single row, 01x06, script generated (kicad-library-utils/schlib/autogen/connector/)")
+    (property "ki_keywords" "connector")
+    (attr through_hole)
+    (fp_text reference "J21" (at 0 -2.77) (layer "F.SilkS")
+        (effects (font (size 1 1) (thickness 0.15)))
+    )
+    (fp_text value "MIC" (at 0 15.47) (layer "F.Fab")
+        (effects (font (size 1 1) (thickness 0.15)))
+    )
+    (fp_text user "${REFERENCE}" (at 0 6.35 90) (layer "F.Fab")
+        (effects (font (size 1 1) (thickness 0.15)))
+    )
+    (fp_line (start -1.33 1.27) (end -1.33 14.03)
+      (stroke (width 0.12) (type solid)) (layer "F.SilkS"))
+    (fp_line (start -1.33 1.27) (end 1.33 1.27)
+      (stroke (width 0.12) (type solid)) (layer "F.SilkS"))
+    (fp_line (start -1.33 14.03) (end 1.33 14.03)
+      (stroke (width 0.12) (type solid)) (layer "F.SilkS"))
+    (fp_line (start 0 -1.33) (end 1.33 -1.33)
+      (stroke (width 0.12) (type solid)) (layer "F.SilkS"))
+    (fp_line (start 1.33 -1.33) (end 1.33 0)
+      (stroke (width 0.12) (type solid)) (layer "F.SilkS"))
+    (fp_line (start 1.33 1.27) (end 1.33 14.03)
+      (stroke (width 0.12) (type solid)) (layer "F.SilkS"))
+    (fp_line (start -1.8 -1.8) (end 1.75 -1.8)
+      (stroke (width 0.05) (type solid)) (layer "F.CrtYd"))
+    (fp_line (start -1.8 14.45) (end -1.8 -1.8)
+      (stroke (width 0.05) (type solid)) (layer "F.CrtYd"))
+    (fp_line (start 1.75 -1.8) (end 1.75 14.45)
+      (stroke (width 0.05) (type solid)) (layer "F.CrtYd"))
+    (fp_line (start 1.75 14.45) (end -1.8 14.45)
+      (stroke (width 0.05) (type solid)) (layer "F.CrtYd"))
+    (fp_line (start -1.27 -1.27) (end 0.635 -1.27)
+      (stroke (width 0.1) (type solid)) (layer "F.Fab"))
+    (fp_line (start -1.27 13.97) (end -1.27 -1.27)
+      (stroke (width 0.1) (type solid)) (layer "F.Fab"))
+    (fp_line (start 0.635 -1.27) (end 1.27 -0.635)
+      (stroke (width 0.1) (type solid)) (layer "F.Fab"))
+    (fp_line (start 1.27 -0.635) (end 1.27 13.97)
+      (stroke (width 0.1) (type solid)) (layer "F.Fab"))
+    (fp_line (start 1.27 13.97) (end -1.27 13.97)
+      (stroke (width 0.1) (type solid)) (layer "F.Fab"))
+    (pad "1" thru_hole rect (at 0 0) (size 1.7 1.7) (drill 1) (layers *.Cu *.Mask)
+      (net 94 "/+3.3v") (pinfunction "Pin_1") (pintype "passive"))
+    (pad "2" thru_hole oval (at 0 2.54) (size 1.7 1.7) (drill 1) (layers *.Cu *.Mask)
+      (net 1 "GND") (pinfunction "Pin_2") (pintype "passive"))
+    (pad "3" thru_hole oval (at 0 5.08) (size 1.7 1.7) (drill 1) (layers *.Cu *.Mask)
+      (net 262 "/CM4_GPIO (GPIO, SDCARD)/BCLK") (pinfunction "Pin_3") (pintype "passive"))
+    (pad "4" thru_hole oval (at 0 7.62) (size 1.7 1.7) (drill 1) (layers *.Cu *.Mask)
+      (net 263 "/CM4_GPIO (GPIO, SDCARD)/DOUT") (pinfunction "Pin_4") (pintype "passive"))
+    (pad "5" thru_hole oval (at 0 10.16) (size 1.7 1.7) (drill 1) (layers *.Cu *.Mask)
+      (net 264 "/CM4_GPIO (GPIO, SDCARD)/LRCL") (pinfunction "Pin_5") (pintype "passive"))
+    (pad "6" thru_hole oval (at 0 12.7) (size 1.7 1.7) (drill 1) (layers *.Cu *.Mask)
+      (net 265 "/CM4_GPIO (GPIO, SDCARD)/SEL") (pinfunction "Pin_6") (pintype "passive"))
+    (model "${KICAD6_3DMODEL_DIR}/Connector_PinSocket_2.54mm.3dshapes/PinSocket_1x06_P2.54mm_Vertical.wrl"
+      (offset (xyz 0 0 0))
+      (scale (xyz 1 1 1))
