File: kicad/USB2-HUB.kicad_sch (KiCad schematic)
At the start: 34 parts

Commit message: Add files via upload
Parts:
- removed U: (no value), symbol CM4IO:TPD4EUSB30
- removed U: (no value), symbol Diode:B340
- renumbered U to C18, U to C19, U to C20, U to C21, U to C22, U to C23, U to C24, U to C25, U to C26, U to C27, U to C28, U to C29, U to C30, U to C31, U to C32, U to J3, U to J4, U to J5, U to J6, U to J7, U to R12, U to R13, U to R14, U to R15, U to R16, U to R17, U to R18, U to R19, U to U3, U to U4, U to U6, U to Y1
Connections:
- net +3.3v: no longer R12.1, R13.2, U3.2 (SEL)
- new net USBOTG: R12.1, R13.2, U3.2 (SEL)
Other:
- note added: "If a cable is plugged into the USB OTG socket CM4 becomes usb device"
- note removed: "If a cable in plugged into the USB C socket CM4 becomes usb device USB can be used to power CM4 (no PCIe)"
- note removed: "Micro USB ESD protection"
- moved on the sheet: C27, C28, C29, C30, C31, C32, J3, J4, J5, J6, J7, R12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

Commit message: Fixing remaining errors
Parts:
- renumbered R13 to U, C29 to U, C30 to U, C31 to U, C32 to U, R12 to U, U6 to U, U4 to U, R16 to U, R15 to U, R14 to U, R19 to U, U3 to U, R17 to U, R18 to U, C24 to U, C25 to U, C26 to U, C22 to U, C20 to U, C21 to U, C18 to U, C19 to U, C23 to U, C27 to U, C28 to U, J3 to U, J7 to U, Y1 to U, J6 to U, J5 to U, J4 to U

Commit message: Mirroring CAM, DSI, new GPDI pinout fix #2 #3 #5 #12
Parts:
- C18, C19: renamed from U; value (none) -> 27pF; footprint (none) -> Capacitor_SMD:C_0402_1005Metric
- C20, C21, C27, C29, C30, C31, C32: renamed from U; value (none) -> 10u; footprint (none) -> Capacitor_SMD:C_0805_2012Metric
- C22, C23, C24, C25, C26: renamed from U; value (none) -> 100n; footprint (none) -> Capacitor_SMD:C_0402_1005Metric
- C28: renamed from U; value (none) -> 100uF; footprint (none) -> Capacitor_Tantalum_SMD:CP_EIA-7132-20_AVX-U
- J3: renamed from U; value (none) -> USB_OTG; footprint (none) -> CM4IO:USB_Micro-B_EDAC_UCON00686
- J4: renamed from U; value (none) -> Conn_01x04_Male; footprint (none) -> Connector_PinHeader_2.00mm:PinHeader_1x04_P2.00mm_Horizontal
- J5, J6: renamed from U; value (none) -> USB_A; footprint (none) -> Connector_USB:USB_A_Molex_67643_Horizontal
- J7: renamed from U; value (none) -> USB_MICRO; footprint (none) -> CM4IO:USB_Micro-B_EDAC_UCON00686
- R12, R13: renamed from U; value (none) -> 2.2K 1%; footprint (none) -> Resistor_SMD:R_0402_1005Metric
- R14, R15, R16, R18: renamed from U; value (none) -> 36K 1%; footprint (none) -> Resistor_SMD:R_0402_1005Metric
- R17: renamed from U; value (none) -> 12K 1%; footprint (none) -> Resistor_SMD:R_0402_1005Metric
- R19: renamed from U; value (none) -> 15K 1%; footprint (none) -> Resistor_SMD:R_0402_1005Metric
- U3: renamed from U; value (none) -> FSUSB42MUX; footprint (none) -> Package_SO:MSOP-10_3x3mm_P0.5mm
- U4: renamed from U; value (none) -> USB2514B-I/M2; footprint (none) -> Package_DFN_QFN:QFN-36-1EP_6x6mm_P0.5mm_EP3.7x3.7mm
- U6: renamed from U; value (none) -> AP22653W6; footprint (none) -> Package_TO_SOT_SMD:SOT-23-6
- Y1: renamed from U; value (none) -> 24MHz; footprint (none) -> Crystal:Crystal_SMD_EuroQuartz_X22-4Pin_2.5x2.0mm_HandSoldering
