File: kicad/CM4_HighSpeed.kicad_sch (KiCad schematic)
At the start: 8 parts

Commit message: Add files via upload
Parts:
- renumbered U to C33, U to C34, U to J10, U to J11, U to J8, U to J9, U to Module1, U to U7
Connections:
- net CAM0_C_N: now also Module1.140 (CAM0_C_N)
- net CAM0_C_P: now also Module1.142 (CAM0_C_P)
- net CAM0_D0_N: now also Module1.128 (CAM0_D0_N)
- net CAM0_D0_P: now also Module1.130 (CAM0_D0_P)
- net CAM0_D1_N: now also Module1.134 (CAM0_D1_N)
- net CAM0_D1_P: now also Module1.136 (CAM0_D1_P)
- net CAM1_C_N: now also Module1.127 (CAM1_C_N)
- net CAM1_C_P: now also Module1.129 (CAM1_C_P)
- net CAM1_D0_N: now also Module1.115 (CAM1_D0_N)
- net CAM1_D0_P: now also Module1.117 (CAM1_D0_P)
- net CAM1_D1_N: now also Module1.121 (CAM1_D1_N)
- net CAM1_D1_P: now also Module1.123 (CAM1_D1_P)
- net CAM1_D2_N: now also Module1.133 (CAM1_D2_N)
- net CAM1_D2_P: now also Module1.135 (CAM1_D2_P)
- net CAM1_D3_N: now also Module1.139 (CAM1_D3_N)
- net CAM1_D3_P: now also Module1.141 (CAM1_D3_P)
- net DSI0_C_N: now also Module1.169 (DSI0_C_N)
- net DSI0_C_P: now also Module1.171 (DSI0_C_P)
- net DSI0_D0_N: now also Module1.157 (DSI0_D0_N)
- net DSI0_D0_P: now also Module1.159 (DSI0_D0_P)
- net DSI0_D1_N: now also Module1.163 (DSI0_D1_N)
- net DSI0_D1_P: now also Module1.165 (DSI0_D1_P)
- net DSI1_C_N: now also Module1.187 (DSI1_C_N)
- net DSI1_C_P: now also Module1.189 (DSI1_C_P)
- net DSI1_D0_N: now also Module1.175 (DSI1_D0_N)
- net DSI1_D0_P: now also Module1.177 (DSI1_D0_P)
- net DSI1_D1_N: now also Module1.181 (DSI1_D1_N)
- net DSI1_D1_P: now also Module1.183 (DSI1_D1_P)
- net DSI1_D2_N: now also Module1.193 (DSI1_D2_N)
- net DSI1_D2_P: now also Module1.195 (DSI1_D2_P)
- net DSI1_D3_N: now also Module1.194 (DSI1_D3_N)
- net DSI1_D3_P: now also Module1.196 (DSI1_D3_P)
- net GND: now also Module1.107 (GND), Module1.108 (GND), Module1.113 (GND), Module1.114 (GND), Module1.119 (GND), Module1.120 (GND), Module1.125 (GND), Module1.126 (GND), Module1.131 (GND), Module1.132 (GND), Module1.137 (GND), Module1.138 (GND), Module1.144 (GND), Module1.150 (GND), Module1.155 (GND), Module1.156 (GND), Module1.161 (GND), Module1.162 (GND), Module1.167 (GND), Module1.168 (GND), Module1.173 (GND), Module1.174 (GND), Module1.179 (GND), Module1.180 (GND), Module1.185 (GND), Module1.186 (GND), Module1.191 (GND), Module1.192 (GND), Module1.197 (GND), Module1.198 (GND)
- net HDMI0_CEC: now also Module1.151 (HDMI0_CEC)
- net HDMI0_CK_N: now also Module1.190 (HDMI0_CLK_N)
- net HDMI0_CK_P: now also Module1.188 (HDMI0_CLK_P)
- net HDMI0_D0_N: now also Module1.184 (HDMI0_TX0_N)
- net HDMI0_D0_P: now also Module1.182 (HDMI0_TX0_P)
- net HDMI0_D1_N: now also Module1.178 (HDMI0_TX1_N)
- net HDMI0_D1_P: now also Module1.176 (HDMI0_TX1_P)
- net HDMI0_D2_N: now also Module1.172 (HDMI0_TX2_N)
- net HDMI0_D2_P: now also Module1.170 (HDMI0_TX2_P)
- net HDMI0_HOTPLUG: now also Module1.153 (HDMI0_HOTPLUG)
- net HDMI0_SCL: now also Module1.200 (HDMI0_SCL)
- net HDMI0_SDA: now also Module1.199 (HDMI0_SDA)
- net HDMI1_CEC: now also Module1.149 (HDMI1_CEC)
- net HDMI1_CK_N: now also Module1.166 (HDMI1_CLK_N)
- net HDMI1_CK_P: now also Module1.164 (HDMI1_CLK_P)
- net HDMI1_D0_N: now also Module1.160 (HDMI1_TX0_N)
- net HDMI1_D0_P: now also Module1.158 (HDMI1_TX0_P)
- net HDMI1_D1_N: now also Module1.154 (HDMI1_TX1_N)
- net HDMI1_D1_P: now also Module1.152 (HDMI1_TX1_P)
- net HDMI1_D2_N: now also Module1.148 (HDMI1_TX2_N)
- net HDMI1_D2_P: now also Module1.146 (HDMI1_TX2_P)
- net HDMI1_HOTPLUG: now also Module1.143 (HDMI1_HOTPLUG)
- net HDMI1_SCL: now also Module1.147 (HDMI1_SCL)
- net HDMI1_SDA: now also Module1.145 (HDMI1_SDA)
- net PCIE_CLK_N: now also Module1.112 (PCIe_CLK_N)
- net PCIE_CLK_P: now also Module1.110 (PCIe_CLK_P)
- net PCIE_CLK_nREQ: now also Module1.102 (PCIe_CLK_nREQ)
- net PCIE_RX_N: now also Module1.118 (PCIe_RX_N)
- net PCIE_RX_P: now also Module1.116 (PCIe_RX_P)
- net PCIE_TX_N: now also Module1.124 (PCIe_TX_N)
- net PCIE_TX_P: now also Module1.122 (PCIe_TX_P)
- net PCIE_nRST: now also Module1.109 (PCIe_nRST)
- net TV_OUT: now also Module1.111 (VDAC_COMP)
- net USB2_N: now also Module1.103 (USB2_N)
- net USB2_P: now also Module1.105 (USB2_P)
- net USBOTG_ID: now also Module1.101 (USB_OTG_ID)

Commit message: Fixing remaining errors
Parts:
- renumbered J8 to U, C34 to U, C33 to U, U7 to U, Module1 to U, J9 to U, J11 to U, J10 to U
Connections:
- net CAM0_C_N: no longer U.140 (CAM0_C_N)
- net CAM0_C_P: no longer U.142 (CAM0_C_P)
- net CAM0_D0_N: no longer U.128 (CAM0_D0_N)
- net CAM0_D0_P: no longer U.130 (CAM0_D0_P)
- net CAM0_D1_N: no longer U.134 (CAM0_D1_N)
- net CAM0_D1_P: no longer U.136 (CAM0_D1_P)
- net CAM1_C_N: no longer U.127 (CAM1_C_N)
- net CAM1_C_P: no longer U.129 (CAM1_C_P)
- net CAM1_D0_N: no longer U.115 (CAM1_D0_N)
- net CAM1_D0_P: no longer U.117 (CAM1_D0_P)
- net CAM1_D1_N: no longer U.121 (CAM1_D1_N)
- net CAM1_D1_P: no longer U.123 (CAM1_D1_P)
- net CAM1_D2_N: no longer U.133 (CAM1_D2_N)
- net CAM1_D2_P: no longer U.135 (CAM1_D2_P)
- net CAM1_D3_N: no longer U.139 (CAM1_D3_N)
- net CAM1_D3_P: no longer U.141 (CAM1_D3_P)
- net DSI0_C_N: no longer U.169 (DSI0_C_N)
- net DSI0_C_P: no longer U.171 (DSI0_C_P)
- net DSI0_D0_N: no longer U.157 (DSI0_D0_N)
- net DSI0_D0_P: no longer U.159 (DSI0_D0_P)
- net DSI0_D1_N: no longer U.163 (DSI0_D1_N)
- net DSI0_D1_P: no longer U.165 (DSI0_D1_P)
- net DSI1_C_N: no longer U.187 (DSI1_C_N)
- net DSI1_C_P: no longer U.189 (DSI1_C_P)
- net DSI1_D0_N: no longer U.175 (DSI1_D0_N)
- net DSI1_D0_P: no longer U.177 (DSI1_D0_P)
- net DSI1_D1_N: no longer U.181 (DSI1_D1_N)
- net DSI1_D1_P: no longer U.183 (DSI1_D1_P)
- net DSI1_D2_N: no longer U.193 (DSI1_D2_N)
- net DSI1_D2_P: no longer U.195 (DSI1_D2_P)
- net DSI1_D3_N: no longer U.194 (DSI1_D3_N)
- net DSI1_D3_P: no longer U.196 (DSI1_D3_P)
- net GND: no longer U.107 (GND), U.108 (GND), U.113 (GND), U.114 (GND), U.119 (GND), U.120 (GND), U.125 (GND), U.126 (GND), U.131 (GND), U.132 (GND), U.137 (GND), U.138 (GND), U.144 (GND), U.150 (GND), U.155 (GND), U.156 (GND), U.161 (GND), U.162 (GND), U.167 (GND), U.168 (GND), U.173 (GND), U.174 (GND), U.179 (GND), U.180 (GND), U.185 (GND), U.186 (GND), U.191 (GND), U.192 (GND), U.197 (GND), U.198 (GND)
- net HDMI0_CEC: no longer U.151 (HDMI0_CEC)
- net HDMI0_CK_N: no longer U.190 (HDMI0_CLK_N)
- net HDMI0_CK_P: no longer U.188 (HDMI0_CLK_P)
- net HDMI0_D0_N: no longer U.184 (HDMI0_TX0_N)
- net HDMI0_D0_P: no longer U.182 (HDMI0_TX0_P)
- net HDMI0_D1_N: no longer U.178 (HDMI0_TX1_N)
- net HDMI0_D1_P: no longer U.176 (HDMI0_TX1_P)
- net HDMI0_D2_N: no longer U.172 (HDMI0_TX2_N)
- net HDMI0_D2_P: no longer U.170 (HDMI0_TX2_P)
- net HDMI0_HOTPLUG: no longer U.153 (HDMI0_HOTPLUG)
- net HDMI0_SCL: no longer U.200 (HDMI0_SCL)
- net HDMI0_SDA: no longer U.199 (HDMI0_SDA)
- net HDMI1_CEC: no longer U.149 (HDMI1_CEC)
- net HDMI1_CK_N: no longer U.166 (HDMI1_CLK_N)
- net HDMI1_CK_P: no longer U.164 (HDMI1_CLK_P)
- net HDMI1_D0_N: no longer U.160 (HDMI1_TX0_N)
- net HDMI1_D0_P: no longer U.158 (HDMI1_TX0_P)
- net HDMI1_D1_N: no longer U.154 (HDMI1_TX1_N)
- net HDMI1_D1_P: no longer U.152 (HDMI1_TX1_P)
- net HDMI1_D2_N: no longer U.148 (HDMI1_TX2_N)
- net HDMI1_D2_P: no longer U.146 (HDMI1_TX2_P)
- net HDMI1_HOTPLUG: no longer U.143 (HDMI1_HOTPLUG)
- net HDMI1_SCL: no longer U.147 (HDMI1_SCL)
- net HDMI1_SDA: no longer U.145 (HDMI1_SDA)
- net PCIE_CLK_N: no longer U.112 (PCIe_CLK_N)
- net PCIE_CLK_P: no longer U.110 (PCIe_CLK_P)
- net PCIE_CLK_nREQ: no longer U.102 (PCIe_CLK_nREQ)
- net PCIE_RX_N: no longer U.118 (PCIe_RX_N)
- net PCIE_RX_P: no longer U.116 (PCIe_RX_P)
- net PCIE_TX_N: no longer U.124 (PCIe_TX_N)
- net PCIE_TX_P: no longer U.122 (PCIe_TX_P)
- net PCIE_nRST: no longer U.109 (PCIe_nRST)
- net TV_OUT: no longer U.111 (VDAC_COMP)
- net USB2_N: no longer U.103 (USB2_N)
- net USB2_P: no longer U.105 (USB2_P)
- net USBOTG_ID: no longer U.101 (USB_OTG_ID)

Commit message: Mirroring CAM, DSI, new GPDI pinout fix #2 #3 #5 #12
Parts:
- removed U (x2): (no value), symbol Connector:HDMI_C_1.4
- added J10: GPDI0, hdmi-d:CONN-10029449-111RLF, symbol hdmi-d:HDMI-D
- added J11: GPDI1, hdmi-d:CONN-10029449-111RLF, symbol hdmi-d:HDMI-D
- added R2: DNP, Resistor_SMD:R_0402_1005Metric, symbol Device:R_Small
- C33, C34: renamed from U; value (none) -> 100n; footprint (none) -> Capacitor_SMD:C_0402_1005Metric
- J8, J9: renamed from U; value (none) -> Conn_01x22_Female; footprint (none) -> Connector_FFC-FPC:Hirose_FH12-22S-0.5SH_1x22-1MP_P0.50mm_Horizontal
- Module1: renamed from U; value (none) -> ComputeModule4; footprint (none) -> CM4IO:Raspberry-Pi-4-Compute-Module-noholes
- U7: renamed from U; value (none) -> RT9742SNGV; footprint (none) -> Package_TO_SOT_SMD:SOT-23
Connections:
- net +3.3v: now also J8.1 (Pin_1), J9.1 (Pin_1); no longer J8.22 (Pin_22), J9.22 (Pin_22)
- net +5v: now also R2.1
- net CAM0_C_N: now also Module1.140 (CAM0_C_N)
- net CAM0_C_P: now also Module1.142 (CAM0_C_P)
- net CAM0_D0_N: now also Module1.128 (CAM0_D0_N)
- net CAM0_D0_P: now also Module1.130 (CAM0_D0_P)
- net CAM0_D1_N: now also Module1.134 (CAM0_D1_N)
- net CAM0_D1_P: now also Module1.136 (CAM0_D1_P)
- net CAM1_C_N: now also J8.15 (Pin_15), Module1.127 (CAM1_C_N); no longer J8.8 (Pin_8)
- net CAM1_C_P: now also J8.14 (Pin_14), Module1.129 (CAM1_C_P); no longer J8.9 (Pin_9)
- net CAM1_D0_N: now also J8.21 (Pin_21), Module1.115 (CAM1_D0_N); no longer J8.2 (Pin_2)
- net CAM1_D0_P: now also J8.20 (Pin_20), Module1.117 (CAM1_D0_P); no longer J8.3 (Pin_3)
- net CAM1_D1_N: now also J8.18 (Pin_18), Module1.121 (CAM1_D1_N); no longer J8.5 (Pin_5)
- net CAM1_D1_P: now also J8.17 (Pin_17), Module1.123 (CAM1_D1_P); no longer J8.6 (Pin_6)
- net CAM1_D2_N: now also J8.12 (Pin_12), Module1.133 (CAM1_D2_N)
- net CAM1_D2_P: now also J8.11 (Pin_11), Module1.135 (CAM1_D2_P)
- net CAM1_D3_N: now also J8.9 (Pin_9), Module1.139 (CAM1_D3_N)
- net CAM1_D3_P: now also J8.8 (Pin_8), Module1.141 (CAM1_D3_P)
- net CAM_GPIO: now also J8.6 (Pin_6); no longer J8.17 (Pin_17)
- net DSI0_C_N: now also Module1.169 (DSI0_C_N)
- net DSI0_C_P: now also Module1.171 (DSI0_C_P)
- net DSI0_D0_N: now also Module1.157 (DSI0_D0_N)
- net DSI0_D0_P: now also Module1.159 (DSI0_D0_P)
- net DSI0_D1_N: now also Module1.163 (DSI0_D1_N)
- net DSI0_D1_P: now also Module1.165 (DSI0_D1_P)
- net DSI1_C_N: now also J9.15 (Pin_15), Module1.187 (DSI1_C_N); no longer J9.8 (Pin_8)
- net DSI1_C_P: now also J9.14 (Pin_14), Module1.189 (DSI1_C_P); no longer J9.9 (Pin_9)
- net DSI1_D0_N: now also J9.21 (Pin_21), Module1.175 (DSI1_D0_N); no longer J9.2 (Pin_2)
- net DSI1_D0_P: now also J9.20 (Pin_20), Module1.177 (DSI1_D0_P); no longer J9.3 (Pin_3)
- net DSI1_D1_N: now also J9.18 (Pin_18), Module1.181 (DSI1_D1_N); no longer J9.5 (Pin_5)
- net DSI1_D1_P: now also J9.17 (Pin_17), Module1.183 (DSI1_D1_P); no longer J9.6 (Pin_6)
- net DSI1_D2_N: now also J9.12 (Pin_12), Module1.193 (DSI1_D2_N); no longer J9.11 (Pin_11)
- net DSI1_D2_P: now also J9.11 (Pin_11), Module1.195 (DSI1_D2_P); no longer J9.12 (Pin_12)
- net DSI1_D3_N: now also J9.9 (Pin_9), Module1.194 (DSI1_D3_N); no longer J9.14 (Pin_14)
- net DSI1_D3_P: now also J9.8 (Pin_8), Module1.196 (DSI1_D3_P); no longer J9.15 (Pin_15)
- net GND: now also J8.22 (Pin_22), J9.22 (Pin_22), Module1.107 (GND), Module1.108 (GND), Module1.113 (GND), Module1.114 (GND), Module1.119 (GND), Module1.120 (GND), Module1.125 (GND), Module1.126 (GND), Module1.131 (GND), Module1.132 (GND), Module1.137 (GND), Module1.138 (GND), Module1.144 (GND), Module1.150 (GND), Module1.155 (GND), Module1.156 (GND), Module1.161 (GND), Module1.162 (GND), Module1.167 (GND), Module1.168 (GND), Module1.173 (GND), Module1.174 (GND), Module1.179 (GND), Module1.180 (GND), Module1.185 (GND), Module1.186 (GND), Module1.191 (GND), Module1.192 (GND), Module1.197 (GND), Module1.198 (GND), J10.0, J10.11 (P11), J10.17 (P17), J10.2 (P2), J10.5 (P5), J10.8 (P8), J11.0, J11.11 (P11), J11.17 (P17), J11.2 (P2), J11.5 (P5), J11.8 (P8); no longer J8.1 (Pin_1), J9.1 (Pin_1)
- net HDMI0_CEC: now also Module1.151 (HDMI0_CEC), J10.13 (P13)
- net HDMI0_CK_N: now also Module1.190 (HDMI0_CLK_N), J10.12 (P12)
- net HDMI0_CK_P: now also Module1.188 (HDMI0_CLK_P), J10.10 (P10)
- net HDMI0_D0_N: now also Module1.184 (HDMI0_TX0_N), J10.9 (P9)
- net HDMI0_D0_P: now also Module1.182 (HDMI0_TX0_P), J10.7 (P7)
- net HDMI0_D1_N: now also Module1.178 (HDMI0_TX1_N), J10.6 (P6)
- net HDMI0_D1_P: now also Module1.176 (HDMI0_TX1_P), J10.4 (P4)
- net HDMI0_D2_N: now also Module1.172 (HDMI0_TX2_N), J10.3 (P3)
- net HDMI0_D2_P: now also Module1.170 (HDMI0_TX2_P), J10.1 (P1)
- net HDMI0_HOTPLUG: now also Module1.153 (HDMI0_HOTPLUG), J10.19 (P19)
- net HDMI0_SCL: now also Module1.200 (HDMI0_SCL), J10.15 (P15)
- net HDMI0_SDA: now also Module1.199 (HDMI0_SDA), J10.16 (P16)
- net HDMI1_CEC: now also Module1.149 (HDMI1_CEC), J11.13 (P13)
- net HDMI1_CK_N: now also Module1.166 (HDMI1_CLK_N), J11.12 (P12)
- net HDMI1_CK_P: now also Module1.164 (HDMI1_CLK_P), J11.10 (P10)
- net HDMI1_D0_N: now also Module1.160 (HDMI1_TX0_N), J11.9 (P9)
- net HDMI1_D0_P: now also Module1.158 (HDMI1_TX0_P), J11.7 (P7)
- net HDMI1_D1_N: now also Module1.154 (HDMI1_TX1_N), J11.6 (P6)
- net HDMI1_D1_P: now also Module1.152 (HDMI1_TX1_P), J11.4 (P4)
- net HDMI1_D2_N: now also Module1.148 (HDMI1_TX2_N), J11.3 (P3)
- net HDMI1_D2_P: now also Module1.146 (HDMI1_TX2_P), J11.1 (P1)
- net HDMI1_HOTPLUG: now also Module1.143 (HDMI1_HOTPLUG), J11.19 (P19)
- net HDMI1_SCL: now also Module1.147 (HDMI1_SCL), J11.15 (P15)
- net HDMI1_SDA: now also Module1.145 (HDMI1_SDA), J11.16 (P16)
- net HDMI_5v: now also J10.18 (P18), J11.18 (P18), R2.2
- net PCIE_CLK_N: now also Module1.112 (PCIe_CLK_N)
- net PCIE_CLK_P: now also Module1.110 (PCIe_CLK_P)
- net PCIE_CLK_nREQ: now also Module1.102 (PCIe_CLK_nREQ)
- net PCIE_RX_N: now also Module1.118 (PCIe_RX_N)
- net PCIE_RX_P: now also Module1.116 (PCIe_RX_P)
- net PCIE_TX_N: now also Module1.124 (PCIe_TX_N)
- net PCIE_TX_P: now also Module1.122 (PCIe_TX_P)
- net PCIE_nRST: now also Module1.109 (PCIe_nRST)
- net SCL0: now also J8.3 (Pin_3), J9.3 (Pin_3); no longer J8.20 (Pin_20), J9.20 (Pin_20)
- net SDA0: now also J8.2 (Pin_2), J9.2 (Pin_2); no longer J8.21 (Pin_21), J9.21 (Pin_21)
- net TV_OUT: now also Module1.111 (VDAC_COMP)
- net USB2_N: now also Module1.103 (USB2_N)
- net USB2_P: now also Module1.105 (USB2_P)
- net USBOTG_ID: now also Module1.101 (USB_OTG_ID)
- no-connect marks 11 -> 7
Other:
- moved on the sheet: C33, C34, U7

Commit message: Adding I2C poullups to schematics
Parts:
- added R34, R35: 4K7, Resistor_SMD:R_0402_1005Metric, symbol Device:R_Small
Connections:
- net +3.3v: now also R34.1, R35.1
- net SCL0: now also R34.2
- net SDA0: now also R35.2
Changed lines of the file:
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@@
     (stroke (width 0) (type solid))
+  )
+  (wire (pts (xy 153.67 163.83) (xy 160.02 163.83))
+    (stroke (width 0) (type default))
   )
   (wire (pts (xy 105.41 133.35) (xy 105.41 140.97))
@@
     (stroke (width 0) (type default))
   )
+  (wire (pts (xy 140.97 163.83) (xy 148.59 163.83))
+    (stroke (width 0) (type default))
+  )
   (wire (pts (xy 102.87 90.17) (xy 119.38 90.17))
     (stroke (width 0) (type solid))
@@
   (wire (pts (xy 39.37 41.91) (xy 41.91 41.91))
     (stroke (width 0) (type solid))
+  )
+  (wire (pts (xy 153.67 156.21) (xy 160.02 156.21))
+    (stroke (width 0) (type default))
   )
   (wire (pts (xy 25.4 143.51) (xy 41.91 143.51))
@@
     (stroke (width 0) (type solid))
   )
+  (wire (pts (xy 140.97 156.21) (xy 148.59 156.21))
+    (stroke (width 0) (type default))
+  )
   (wire (pts (xy 163.83 124.46) (xy 166.37 124.46))
     (stroke (width 0) (type solid))
@@
     (effects (font (size 1.27 1.27)) (justify left bottom))
   )
+  (label "SDA0" (at 160.02 163.83 0) (fields_autoplaced)
+    (effects (font (size 1.27 1.27)) (justify right bottom))
+  )
   (label "DSI1_C_P" (at 189.23 48.26 0) (fields_autoplaced)
     (effects (font (size 1.27 1.27)) (justify left bottom))
@@
     (effects (font (size 1.27 1.27)) (justify right bottom))
   )
+  (label "+3.3v" (at 140.97 163.83 0) (fields_autoplaced)
+    (effects (font (size 1.27 1.27)) (justify left bottom))
+  )
   (label "HDMI1_D1_P" (at 25.4 90.17 0) (fields_autoplaced)
     (effects (font (size 1.27 1.27)) (justify left bottom))
@@
     (effects (font (size 1.27 1.27)) (justify left bottom))
   )
+  (label "+3.3v" (at 140.97 156.21 0) (fields_autoplaced)
+    (effects (font (size 1.27 1.27)) (justify left bottom))
+  )
   (label "HDMI0_D1_P" (at 25.4 120.65 0) (fields_autoplaced)
     (effects (font (size 1.27 1.27)) (justify left bottom))
@@
   (label "DSI1_C_N" (at 189.23 45.72 0) (fields_autoplaced)
     (effects (font (size 1.27 1.27)) (justify left bottom))
+  )
+  (label "SCL0" (at 160.02 156.21 0) (fields_autoplaced)
+    (effects (font (size 1.27 1.27)) (justify right bottom))
   )
   (label "DSI1_D0_P" (at 119.38 123.19 0) (fields_autoplaced)
@@
     )
   )
+  (symbol (lib_id "Device:R_Small") (at 151.13 156.21 90) (unit 1)
+    (in_bom yes) (on_board yes) (dnp no) (fields_autoplaced)
+    (property "Reference" "R34" (at 151.13 151.13 90)
+      (effects (font (size 1.27 1.27)))
+    )
+    (property "Value" "4K7" (at 151.13 153.67 90)
+      (effects (font (size 1.27 1.27)))
+    )
+    (property "Footprint" "Resistor_SMD:R_0402_1005Metric" (at 151.13 156.21 0)
+      (effects (font (size 1.27 1.27)) hide)
+    )
+    (property "Datasheet" "~" (at 151.13 156.21 0)
+      (effects (font (size 1.27 1.27)) hide)
+    )
+    (pin "1")
+    (pin "2")
+    (instances
+      (project "Unifying"
+        (path "/9bdfb27f-c9ad-4974-8286-b25e5ffa2770/00000000-0000-0000-0000-00005cff70b1"
+          (reference "R34") (unit 1) (value "4K7") (footprint "Resistor_SMD:R_0402_1005Metric")
+        )
+      )
+    )
+  )
   (symbol (lib_id "Device:R_Small") (at 156.21 113.03 90) (unit 1)
     (in_bom yes) (on_board yes) (dnp no) (fields_autoplaced)
@@
         )
       )
+    )
+  )
+  (symbol (lib_id "Device:R_Small") (at 151.13 163.83 90) (unit 1)
+    (in_bom yes) (on_board yes) (dnp no) (fields_autoplaced)
+    (property "Reference" "R35" (at 151.13 158.75 90)
+      (effects (font (size 1.27 1.27)))
+    )
+    (property "Value" "4K7" (at 151.13 161.29 90)
+      (effects (font (size 1.27 1.27)))
+    )
+    (property "Footprint" "Resistor_SMD:R_0402_1005Metric" (at 151.13 163.83 0)
+      (effects (font (size 1.27 1.27)) hide)
+    )
+    (property "Datasheet" "~" (at 151.13 163.83 0)
+      (effects (font (size 1.27 1.27)) hide)
+    )
+    (pin "1")
+    (pin "2")
+    (instances
+      (project "Unifying"
+        (path "/9bdfb27f-c9ad-4974-8286-b25e5ffa2770/00000000-0000-0000-0000-00005cff70b1"
+          (reference "R35") (unit 1) (value "4K7") (footprint "Resistor_SMD:R_0402_1005Metric")
+        )
+      )
